File: system_design/Georgetown/V0.5.2/EDA/main_board/main_board.kicad_pcb (KiCad board)
At the start: 2 copper layers, 40.6 x 82.6 mm, 36 parts, among them J1 B3B-XH-A_LF__SN_, J2 Conn_01x02_Pin, P1 SD card socket, Q1 MMBT2222A, SW1 SW_Wuerth_450301014042, U1 HX-2S-JH10, U2 DS3231M, U4 BME280_module, U5 KA78M05_TO252

Commit message: PCB gerber created
Other:
- board text added: "06/01/2026"
- board text added: "B"
- board text added: "DS3231M"
- board text added: "R"
- board text added: "Stage Height V0.5.2"
- board text added: "Y"
- board text removed: "Amanda Sark"
- board text removed: "DS3231"
- board text removed: "Stage Height V0.5.1"
Changed lines of the file:
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@@
 			(drillshape 0)
 			(scaleselection 1)
-			(outputdirectory "../Gerber files/")
+			(outputdirectory "../UAV-Deployable-Stage-Height-Sensor V0.5.2 - Gerber files/")
 		)
 	)
@@
 		)
 		(property "Value" "Arduino_Nano_v2.x-MCU_Module"
-			(at 8.89 19.05 90)
+			(at 7.45 30.89 90)
 			(layer "F.Fab")
 			(effects
@@
 		)
 		(fp_text user "${REFERENCE}"
-			(at 6.35 19.05 90)
+			(at 5.25 25.9 90)
 			(layer "F.Fab")
 			(effects
@@
 		(tags "SOT TO_SOT_SMD")
 		(property "Reference" "Q1"
-			(at -1.13 -2.67 0)
+			(at 2.13 1.61 0)
 			(layer "F.SilkS")
 			(effects
@@
 		(at 171.3 82.1 -90)
 		(property "Reference" "BT1"
-			(at 0 -5.5 90)
+			(at -7.3 -3.71 90)
 			(layer "F.SilkS")
 			(effects
@@
 		)
 		(property "Value" "Battery_Cell"
-			(at 0 -9.525 90)
+			(at -0.14 -1.36 90)
 			(layer "F.Fab")
 			(effects
@@
 		(tags "capacitor handsolder")
 		(property "Reference" "R3"
-			(at 0.13 1.94 0)
+			(at -0.25 -2.1 0)
 			(layer "F.SilkS")
 			(effects
@@
 		(at 167.68 109.875 180)
 		(property "Reference" "U3"
-			(at 0 -11.43 0)
+			(at 0 -11.43 180)
 			(unlocked yes)
-			(layer "B.SilkS")
+			(layer "F.SilkS")
 			(effects
 				(font
@@
 					(thickness 0.1)
 				)
-				(justify mirror)
 			)
 		)
@@
 		(at 157.99 146.33 180)
 		(property "Reference" "Ultrasonic_sensor1"
-			(at 0 -2.67 0)
+			(at 12.47 -2.12 0)
 			(layer "B.SilkS")
 			(effects
@@
 		(at 167.43 79.48 -90)
 		(property "Reference" "P1"
-			(at 10.52 1.43 90)
+			(at 6.53 7.22 0)
 			(layer "B.SilkS")
 			(effects
@@
 		)
 	)
-	(gr_text "Stage Height V0.5.1"
-		(at 139.5 132 90)
+	(gr_text "B"
+		(at 173.33 147.85 0)
+		(layer "F.SilkS")
+		(effects
+			(font
+				(size 1 1)
+				(thickness 0.15)
+			)
+		)
+	)
+	(gr_text "R"
+		(at 168.27 147.99 0)
+		(layer "F.SilkS")
+		(effects
+			(font
+				(size 1 1)
+				(thickness 0.15)
+			)
+		)
+	)
+	(gr_text "Stage Height V0.5.2"
+		(at 157.85 68.89 0)
 		(layer "F.SilkS")
 		(effects
@@
 	)
 	(gr_text "Arduino Nano"
-		(at 152 114.5 90)
+		(at 153.95 127.82 90)
 		(layer "F.SilkS")
 		(effects
@@
 		)
 	)
-	(gr_text "DS3231"
+	(gr_text "DS3231M"
 		(at 139 84.5 90)
 		(layer "F.SilkS")
@@
 		)
 	)
+	(gr_text "Y"
+		(at 170.8 147.92 0)
+		(layer "F.SilkS")
+		(effects
+			(font
+				(size 1 1)
+				(thickness 0.15)
+			)
+		)
+	)
 	(gr_text "LED"
 		(at 143 98 0)
@@
 		)
 	)
+	(gr_text "06/01/2026"
+		(at 158.09 68.79 0)
+		(layer "B.SilkS")
+		(effects
+			(font
+				(size 1.3 1.3)
+				(thickness 0.2)
+			)
+			(justify mirror)
+		)
+	)
 	(gr_text "BME"
 		(at 141 141.5 90)
@@
 		(layer "B.SilkS")
 		(effects
-			(font
-				(size 1.000504 1.000504)
-				(thickness 0.15)
-			)
-			(justify mirror)
-		)
-	)
-	(gr_text "Amanda Sark"
-		(at 171.4 96.5 0)
-		(layer "B.SilkS")
-		(effects
